Commit message: added absolute paths to xacro for meshes

File: install/echo_sim_v1/share/echo_sim_v1/urdf/echo_v1.urdf.xacro (robot description, xacro)
@@ -1,4 +1,6 @@
 <?xml version="1.0" encoding="utf-8"?>
 <robot name="echo_v1" xmlns:xacro="http://ros.org/wiki/xacro">
+  <!-- Include mesh directory env variable -->
+  <xacro:property name="mesh_dir" value="$(env HOME)/Project_Echo/Educational/amr_ws/src/echo_sim_v1/meshes"/>
   <!-- Include materials xacro -->
   <xacro:include filename="$(find echo_sim_v1)/urdf/materials.xacro"/>
@@ -21,5 +23,5 @@
       <origin xyz="0 0 0" rpy="0 0 0"/>
       <geometry>
-        <mesh filename="package://echo_sim_v1/meshes/base_link.STL"/>
+        <mesh filename="${mesh_dir}/base_link.STL"/>
       </geometry>
       <material name="red"/>
@@ -35,5 +37,5 @@
       <origin xyz="0 0 0" rpy="0 0 0"/>
       <geometry>
-        <mesh filename="package://echo_sim_v1/meshes/base_link.STL"/>
+        <mesh filename="${mesh_dir}/base_link.STL"/>
       </geometry>
     </collision>
@@ -50,5 +52,5 @@
       <origin xyz="0 0 0" rpy="0 0 0"/>
       <geometry>
-        <mesh filename="package://echo_sim_v1/meshes/left_wheel_link.STL"/>
+        <mesh filename="${mesh_dir}/left_wheel_link.STL"/>
       </geometry>
       <material name="silver"/>
@@ -57,5 +59,5 @@
       <origin xyz="0 0 0" rpy="0 0 0"/>
       <geometry>
-        <mesh filename="package://echo_sim_v1/meshes/left_wheel_link.STL"/>
+        <mesh filename="${mesh_dir}/left_wheel_link.STL"/>
       </geometry>
     </collision>
@@ -78,5 +80,5 @@
       <origin xyz="0 0 0" rpy="0 0 0"/>
       <geometry>
-        <mesh filename="package://echo_sim_v1/meshes/right_wheel_link.STL"/>
+        <mesh filename="${mesh_dir}/right_wheel_link.STL"/>
       </geometry>
       <material name="silver"/>
@@ -85,5 +87,5 @@
       <origin xyz="0 0 0" rpy="0 0 0"/>
       <geometry>
-        <mesh filename="package://echo_sim_v1/meshes/right_wheel_link.STL"/>
+        <mesh filename="${mesh_dir}/right_wheel_link.STL"/>
       </geometry>
     </collision>
@@ -106,5 +108,5 @@
       <origin xyz="0 0 0" rpy="0 0 0"/>
       <geometry>
-        <mesh filename="package://echo_sim_v1/meshes/caster_wheel_link.STL"/>
+        <mesh filename="${mesh_dir}/caster_wheel_link.STL"/>
       </geometry>
       <material name="silver"/>
@@ -113,5 +115,5 @@
       <origin xyz="0 0 0" rpy="0 0 0"/>
       <geometry>
-        <mesh filename="package://echo_sim_v1/meshes/caster_wheel_link.STL"/>
+        <mesh filename="${mesh_dir}/caster_wheel_link.STL"/>
       </geometry>
     </collision>
@@ -134,5 +136,5 @@
       <origin xyz="0 0 0" rpy="0 0 0"/>
       <geometry>
-        <mesh filename="package://echo_sim_v1/meshes/lidar_link.STL"/>
+        <mesh filename="${mesh_dir}/lidar_link.STL"/>
       </geometry>
       <material name="dark_grey"/>
@@ -141,5 +143,5 @@
       <origin xyz="0 0 0" rpy="0 0 0"/>
       <geometry>
-        <mesh filename="package://echo_sim_v1/meshes/lidar_link.STL"/>
+        <mesh filename="${mesh_dir}/lidar_link.STL"/>
       </geometry>
     </collision>
@@ -162,5 +164,5 @@
       <origin xyz="0 0 0" rpy="0 0 0"/>
       <geometry>
-        <mesh filename="package://echo_sim_v1/meshes/camera_link.STL"/>
+        <mesh filename="${mesh_dir}/camera_link.STL"/>
       </geometry>
       <material name="dark_grey"/>
@@ -169,5 +171,5 @@
       <origin xyz="0 0 0" rpy="0 0 0"/>
       <geometry>
-        <mesh filename="package://echo_sim_v1/meshes/camera_link.STL"/>
+        <mesh filename="${mesh_dir}/camera_link.STL"/>
       </geometry>
     </collision>

Commit message: changes to project layout

File: install/echo_sim_v1/share/echo_sim_v1/urdf/echo_v1.urdf.xacro (robot description, xacro)
@@ -5,4 +5,35 @@
   <!-- Include materials xacro -->
   <xacro:include filename="$(find echo_sim_v1)/urdf/materials.xacro"/>
+  <!-- ROS2 Control Plugin -->
+  <ros2_control name="EchoHardware" type="system">
+    <hardware>
+      <plugin>gazebo_ros2_control/GazeboSystem</plugin>
+    </hardware>
+    <joint name="left_wheel_joint">
+      <command_interface name="velocity"/>
+      <state_interface name="velocity"/>
+      <state_interface name="position"/>
+    </joint>
+    <joint name="right_wheel_joint">
+      <command_interface name="velocity"/>
+      <state_interface name="velocity"/>
+      <state_interface name="position"/>
+    </joint>
+  </ros2_control>
+  <!-- Transmission Definition -->
+  <transmission name="left_wheel_trans">
+    <type>transmission_interface/SimpleTransmission</type>
+    <actuator name="left_wheel_motor">
+      <mechanicalReduction>1</mechanicalReduction>
+    </actuator>
+    <joint name="left_wheel_joint"/>
+  </transmission>
+  <transmission name="right_wheel_trans">
+    <type>transmission_interface/SimpleTransmission</type>
+    <actuator name="right_wheel_motor">
+      <mechanicalReduction>1</mechanicalReduction>
+    </actuator>
+    <joint name="right_wheel_joint"/>
+  </transmission>
   <!-- Base Footprint -->
   <link name="base_footprint"/>

File: src/echo_sim_v1/urdf/echo_v1.urdf.xacro (robot description, xacro)
@@ -5,18 +5,35 @@
   <!-- Include materials xacro -->
   <xacro:include filename="$(find echo_sim_v1)/urdf/materials.xacro"/>
-  <!-- Diff Drive Plugin for Gazebo -->
-  <gazebo>
-    <plugin name="diff_drive_controller" filename="libgazebo_ros_diff_drive.so">
-      <ros>
-        <namespace>/</namespace>
-      </ros>
-      <command_topic>/cmd_vel</command_topic>
-      <left_wheel>left_wheel_joint</left_wheel>
-      <right_wheel>right_wheel_joint</right_wheel>
-      <wheel_separation>0.14</wheel_separation>
-      <wheel_radius>0.03</wheel_radius>
-      <publish_wheel_tf>true</publish_wheel_tf>
-    </plugin>
-  </gazebo>
+  <!-- ROS2 Control Plugin -->
+  <ros2_control name="EchoHardware" type="system">
+    <hardware>
+      <plugin>gazebo_ros2_control/GazeboSystem</plugin>
+    </hardware>
+    <joint name="left_wheel_joint">
+      <command_interface name="velocity"/>
+      <state_interface name="velocity"/>
+      <state_interface name="position"/>
+    </joint>
+    <joint name="right_wheel_joint">
+      <command_interface name="velocity"/>
+      <state_interface name="velocity"/>
+      <state_interface name="position"/>
+    </joint>
+  </ros2_control>
+  <!-- Transmission Definition -->
+  <transmission name="left_wheel_trans">
+    <type>transmission_interface/SimpleTransmission</type>
+    <actuator name="left_wheel_motor">
+      <mechanicalReduction>1</mechanicalReduction>
+    </actuator>
+    <joint name="left_wheel_joint"/>
+  </transmission>
+  <transmission name="right_wheel_trans">
+    <type>transmission_interface/SimpleTransmission</type>
+    <actuator name="right_wheel_motor">
+      <mechanicalReduction>1</mechanicalReduction>
+    </actuator>
+    <joint name="right_wheel_joint"/>
+  </transmission>
   <!-- Base Footprint -->
   <link name="base_footprint"/>

Commit message: fixed urdf filepath for rviz

File: install/echo_sim_v1/share/echo_sim_v1/urdf/echo_v1.urdf.xacro (robot description, xacro)
@@ -1,9 +1,7 @@
 <?xml version="1.0" encoding="utf-8"?>
 <robot name="echo_v1" xmlns:xacro="http://ros.org/wiki/xacro">
-  <!-- Include mesh directory env variable -->
-  <xacro:property name="mesh_dir" value="$(env HOME)/Project_Echo/Educational/amr_ws/src/echo_sim_v1/meshes"/>
   <!-- Include materials xacro -->
-  <xacro:include filename="$(find echo_sim_v1)/urdf/materials.xacro"/>
-  <!-- ROS2 Control Plugin -->
+  <xacro:include filename="/home/cameron/Project_Echo/Educational/amr_ws/src/echo_sim_v1/urdf/materials.xacro"/>
+  <!-- ROS2 Control Plugin
   <ros2_control name="EchoHardware" type="system">
     <hardware>
@@ -20,7 +18,7 @@
       <state_interface name="position"/>
     </joint>
-  </ros2_control>
+  </ros2_control> -->
   <!-- Transmission Definition -->
-  <transmission name="left_wheel_trans">
+  <!-- <transmission name="left_wheel_trans">
     <type>transmission_interface/SimpleTransmission</type>
     <actuator name="left_wheel_motor">
@@ -35,5 +33,5 @@
     </actuator>
     <joint name="right_wheel_joint"/>
-  </transmission>
+  </transmission> -->
   <!-- Base Footprint -->
   <link name="base_footprint"/>
@@ -54,22 +52,16 @@
       <origin xyz="0 0 0" rpy="0 0 0"/>
       <geometry>
-        <mesh filename="${mesh_dir}/base_link.STL"/>
+        <mesh filename="file:///home/cameron/Project_Echo/Educational/amr_ws/src/echo_sim_v1/meshes/base_link.STL"/>
       </geometry>
       <material name="red"/>
     </visual>
-    <!-- <visual>
-      <origin xyz="0 0 0" rpy="0 0 0" />
-      <geometry>
-       <box size="0.3 0.3 0.1"/>
-      </geometry>
-      <material name="Red"/>
-    </visual> -->
-    <collision>
-      <origin xyz="0 0 0" rpy="0 0 0"/>
-      <geometry>
-        <mesh filename="${mesh_dir}/base_link.STL"/>
-      </geometry>
-    </collision>
-  </link>
+    <collision>
+      <origin xyz="0 0 0" rpy="0 0 0"/>
+      <geometry>
+        <mesh filename="file:///home/cameron/Project_Echo/Educational/amr_ws/src/echo_sim_v1/meshes/base_link.STL"/>
+      </geometry>
+    </collision>
+  </link>
+W
   <!-- Left Wheel -->
   <link name="left_wheel_link">
@@ -83,5 +75,5 @@
       <origin xyz="0 0 0" rpy="0 0 0"/>
       <geometry>
-        <mesh filename="${mesh_dir}/left_wheel_link.STL"/>
+        <mesh filename="file:///home/cameron/Project_Echo/Educational/amr_ws/src/echo_sim_v1/meshes/left_wheel_link.STL"/>
       </geometry>
       <material name="silver"/>
@@ -90,5 +82,5 @@
       <origin xyz="0 0 0" rpy="0 0 0"/>
       <geometry>
-        <mesh filename="${mesh_dir}/left_wheel_link.STL"/>
+        <mesh filename="file:///home/cameron/Project_Echo/Educational/amr_ws/src/echo_sim_v1/meshes/left_wheel_link.STL"/>
       </geometry>
     </collision>
@@ -111,5 +103,5 @@
       <origin xyz="0 0 0" rpy="0 0 0"/>
       <geometry>
-        <mesh filename="${mesh_dir}/right_wheel_link.STL"/>
+        <mesh filename="file:///home/cameron/Project_Echo/Educational/amr_ws/src/echo_sim_v1/meshes/right_wheel_link.STL"/>
       </geometry>
       <material name="silver"/>
@@ -118,5 +110,5 @@
       <origin xyz="0 0 0" rpy="0 0 0"/>
       <geometry>
-        <mesh filename="${mesh_dir}/right_wheel_link.STL"/>
+        <mesh filename="file:///home/cameron/Project_Echo/Educational/amr_ws/src/echo_sim_v1/meshes/right_wheel_link.STL"/>
       </geometry>
     </collision>
@@ -139,5 +131,5 @@
       <origin xyz="0 0 0" rpy="0 0 0"/>
       <geometry>
-        <mesh filename="${mesh_dir}/caster_wheel_link.STL"/>
+        <mesh filename="file:///home/cameron/Project_Echo/Educational/amr_ws/src/echo_sim_v1/meshes/caster_wheel_link.STL"/>
       </geometry>
       <material name="silver"/>
@@ -146,5 +138,5 @@
       <origin xyz="0 0 0" rpy="0 0 0"/>
       <geometry>
-        <mesh filename="${mesh_dir}/caster_wheel_link.STL"/>
+        <mesh filename="file:///home/cameron/Project_Echo/Educational/amr_ws/src/echo_sim_v1/meshes/caster_wheel_link.STL"/>
       </geometry>
     </collision>
@@ -167,5 +159,5 @@
       <origin xyz="0 0 0" rpy="0 0 0"/>
       <geometry>
-        <mesh filename="${mesh_dir}/lidar_link.STL"/>
+        <mesh filename="file:///home/cameron/Project_Echo/Educational/amr_ws/src/echo_sim_v1/meshes/lidar_link.STL"/>
       </geometry>
       <material name="dark_grey"/>
@@ -174,5 +166,5 @@
       <origin xyz="0 0 0" rpy="0 0 0"/>
       <geometry>
-        <mesh filename="${mesh_dir}/lidar_link.STL"/>
+        <mesh filename="file:///home/cameron/Project_Echo/Educational/amr_ws/src/echo_sim_v1/meshes/lidar_link.STL"/>
       </geometry>
     </collision>
@@ -195,5 +187,5 @@
       <origin xyz="0 0 0" rpy="0 0 0"/>
       <geometry>
-        <mesh filename="${mesh_dir}/camera_link.STL"/>
+        <mesh filename="file:///home/cameron/Project_Echo/Educational/amr_ws/src/echo_sim_v1/meshes/camera_link.STL"/>
       </geometry>
       <material name="dark_grey"/>
@@ -202,5 +194,5 @@
       <origin xyz="0 0 0" rpy="0 0 0"/>
       <geometry>
-        <mesh filename="${mesh_dir}/camera_link.STL"/>
+        <mesh filename="file:///home/cameron/Project_Echo/Educational/amr_ws/src/echo_sim_v1/meshes/camera_link.STL"/>
       </geometry>
     </collision>
