Commit message: lots of additions

File: install/echo_sim_v1/share/echo_sim_v1/urdf/echo_v1.urdf.xacro (robot description, xacro)
@@ -1,206 +1,175 @@
 <?xml version="1.0" encoding="utf-8"?>
-<robot name="echo_v1" xmlns:xacro="http://ros.org/wiki/xacro">
-  <!-- Include materials xacro -->
+<robot name="echo_v1" xmlns:xacro="http://www.ros.org/wiki/xacro">
+  <!-- ========================= -->
+  <!-- Global Properties & Macros -->
+  <!-- ========================= -->
+<!-- Include  gazebo control xacro -->
+  <xacro:include filename="/home/cameron/Project_Echo/Educational/amr_ws/src/echo_sim_v1/urdf/gazebo_control.xacro"/>
+<!-- Include materials xacro -->
   <xacro:include filename="/home/cameron/Project_Echo/Educational/amr_ws/src/echo_sim_v1/urdf/materials.xacro"/>
-  <!-- ROS2 Control Plugin
-  <ros2_control name="EchoHardware" type="system">
-    <hardware>
-      <plugin>gazebo_ros2_control/GazeboSystem</plugin>
-    </hardware>
-    <joint name="left_wheel_joint">
-      <command_interface name="velocity"/>
-      <state_interface name="velocity"/>
-      <state_interface name="position"/>
-    </joint>
-    <joint name="right_wheel_joint">
-      <command_interface name="velocity"/>
-      <state_interface name="velocity"/>
-      <state_interface name="position"/>
-    </joint>
-  </ros2_control> -->
-  <!-- Transmission Definition -->
-  <!-- <transmission name="left_wheel_trans">
-    <type>transmission_interface/SimpleTransmission</type>
-    <actuator name="left_wheel_motor">
-      <mechanicalReduction>1</mechanicalReduction>
-    </actuator>
-    <joint name="left_wheel_joint"/>
-  </transmission>
-  <transmission name="right_wheel_trans">
-    <type>transmission_interface/SimpleTransmission</type>
-    <actuator name="right_wheel_motor">
-      <mechanicalReduction>1</mechanicalReduction>
-    </actuator>
-    <joint name="right_wheel_joint"/>
-  </transmission> -->
-  <!-- Base Footprint -->
-  <link name="base_footprint"/>
-  <joint name="base_footprint_to_base_link" type="fixed">
-    <origin xyz="0 0 0.02" rpy="-1.5708 0 0"/>
-    <parent link="base_footprint"/>
-    <child link="base_link"/>
+<!-- Include lidar xacro -->
+  <xacro:include filename="/home/cameron/Project_Echo/Educational/amr_ws/src/echo_sim_v1/urdf/lidar.xacro"/>
+  <!-- Inertia Macros -->
+  <xacro:macro name="inertial_sphere" params="mass radius *origin">
+    <inertial>
+      <xacro:insert_block name="origin"/>
+      <mass value="${mass}" />
+      <inertia ixx="${(2/5) * mass * (radius*radius)}" ixy="0.0" ixz="0.0"
+               iyy="${(2/5) * mass * (radius*radius)}" iyz="0.0"
+               izz="${(2/5) * mass * (radius*radius)}" />
+    </inertial>
+  </xacro:macro>
+  <xacro:macro name="inertial_box" params="mass x y z *origin">
+    <inertial>
+      <xacro:insert_block name="origin"/>
+      <mass value="${mass}" />
+      <inertia ixx="${(1/12) * mass * (y*y+z*z)}" ixy="0.0" ixz="0.0"
+               iyy="${(1/12) * mass * (x*x+z*z)}" iyz="0.0"
+               izz="${(1/12) * mass * (x*x+y*y)}" />
+    </inertial>
+  </xacro:macro>
+  <xacro:macro name="inertial_cylinder" params="mass length radius *origin">
+    <inertial>
+      <xacro:insert_block name="origin"/>
+      <mass value="${mass}" />
+      <inertia ixx="${(1/12) * mass * (3*radius*radius + length*length)}" ixy="0.0" ixz="0.0"
+               iyy="${(1/12) * mass * (3*radius*radius + length*length)}" iyz="0.0"
+               izz="${(1/2) * mass * (radius*radius)}" />
+    </inertial>
+  </xacro:macro>
+  <!-- ========================= -->
+  <!-- Links and Joints -->
+  <!-- ========================= -->
+  <!-- Base link (empty root) -->
+  <link name="base_link"/>
+  <!-- Chassis -->
+  <joint name="chassis_joint" type="fixed">
+    <parent link="base_link"/>
+    <child link="chassis"/>
+    <origin xyz="-0.1 0 0"/>
   </joint>
-  <!-- Base Link -->
-  <link name="base_link">
-    <inertial>
-      <origin xyz="0.00088588 5.7031E-05 0.02478" rpy="0 0 0"/>
-      <mass value="0.99833"/>
-      <inertia ixx="0.0010305" ixy="-1.7168E-06" ixz="1.5313E-05"
-               iyy="0.0035021" iyz="1.7459E-07" izz="0.0041088"/>
-    </inertial>
+  <link name="chassis">
     <visual>
-      <origin xyz="0 0 0" rpy="0 0 0"/>
+      <origin xyz="0.15 0 0.075"/>
       <geometry>
-        <mesh filename="file:///home/cameron/Project_Echo/Educational/amr_ws/src/echo_sim_v1/meshes/base_link.STL"/>
+        <box size="0.4 0.3 0.1"/>
       </geometry>
       <material name="red"/>
     </visual>
     <collision>
-      <origin xyz="0 0 0" rpy="0 0 0"/>
+      <origin xyz="0.15 0 0.075"/>
       <geometry>
-        <mesh filename="file:///home/cameron/Project_Echo/Educational/amr_ws/src/echo_sim_v1/meshes/base_link.STL"/>
+        <box size="0.4 0.3 0.1"/>
       </geometry>
     </collision>
+    <xacro:inertial_box mass="0.5" x="0.4" y="0.3" z="0.1">
+      <origin xyz="0.15 0 0.075" rpy="0 0 0"/>
+    </xacro:inertial_box>
   </link>
-W
+  <gazebo reference="chassis">
+    <material>Gazebo/Red</material>
+  </gazebo>
   <!-- Left Wheel -->
-  <link name="left_wheel_link">
-    <inertial>
-      <origin xyz="-1.3878E-17 0.0075 0" rpy="0 0 0"/>
-      <mass value="0.073711"/>
-      <inertia ixx="3.0207E-05" ixy="-3.1866E-38" ixz="1.075E-37"
-               iyy="5.7735E-05" iyz="1.0613E-38" izz="3.0207E-05"/>
-    </inertial>
+  <joint name="left_wheel_joint" type="continuous">
+    <parent link="base_link"/>
+    <child link="left_wheel"/>
+    <origin xyz="-0.07 0.175 0" rpy="-${pi/2} 0 0"/>
+    <axis xyz="0 0 1"/>
+  </joint>
+  <link name="left_wheel">
     <visual>
-      <origin xyz="0 0 0" rpy="0 0 0"/>
       <geometry>
-        <mesh filename="file:///home/cameron/Project_Echo/Educational/amr_ws/src/echo_sim_v1/meshes/left_wheel_link.STL"/>
-      </geometry>
-      <material name="silver"/>
-    </visual>
-    <collision>
-      <origin xyz="0 0 0" rpy="0 0 0"/>
-      <geometry>
-        <mesh filename="file:///home/cameron/Project_Echo/Educational/amr_ws/src/echo_sim_v1/meshes/left_wheel_link.STL"/>
-      </geometry>
-    </collision>
-  </link>
-  <joint name="base_link_to_left_wheel" type="continuous">
-    <origin xyz="-0.07 -0.02 0.05" rpy="-1.5708 0 -1.5708"/>
-    <parent link="base_link"/>
-    <child link="left_wheel_link"/>
-    <axis xyz="0 -1 0"/>
-  </joint>
-  <!-- Right Wheel -->
-  <link name="right_wheel_link">
-    <inertial>
-      <origin xyz="-1.3878E-17 -0.0075 0" rpy="0 0 0"/>
-      <mass value="0.073711"/>
-      <inertia ixx="3.0207E-05" ixy="-3.1866E-38" ixz="1.075E-37"
-               iyy="5.7735E-05" iyz="1.0613E-38" izz="3.0207E-05"/>
-    </inertial>
-    <visual>
-      <origin xyz="0 0 0" rpy="0 0 0"/>
-      <geometry>
-        <mesh filename="file:///home/cameron/Project_Echo/Educational/amr_ws/src/echo_sim_v1/meshes/right_wheel_link.STL"/>
-      </geometry>
-      <material name="silver"/>
-    </visual>
-    <collision>
-      <origin xyz="0 0 0" rpy="0 0 0"/>
-      <geometry>
-        <mesh filename="file:///home/cameron/Project_Echo/Educational/amr_ws/src/echo_sim_v1/meshes/right_wheel_link.STL"/>
-      </geometry>
-    </collision>
-  </link>
-  <joint name="base_link_to_right_wheel" type="continuous">
-    <origin xyz="-0.07 -0.02 -0.05" rpy="1.5708 0 0"/>
-    <parent link="base_link"/>
-    <child link="right_wheel_link"/>
-    <axis xyz="0 1 0"/>
-  </joint>
-  <!-- Caster Wheel -->
-  <link name="caster_wheel_link">
-    <inertial>
-      <origin xyz="1.3878E-17 -5.5511E-17 0.0045" rpy="0 0 0"/>
-      <mass value="0.0036191"/>
-      <inertia ixx="1.3517E-07" ixy="-1.3235E-23" ixz="-8.7993E-24"
-               iyy="1.3517E-07" iyz="-5.2645E-22" izz="2.0846E-07"/>
-    </inertial>
-    <visual>
-      <origin xyz="0 0 0" rpy="0 0 0"/>
-      <geometry>
-        <mesh filename="file:///home/cameron/Project_Echo/Educational/amr_ws/src/echo_sim_v1/meshes/caster_wheel_link.STL"/>
-      </geometry>
-      <material name="silver"/>
-    </visual>
-    <collision>
-      <origin xyz="0 0 0" rpy="0 0 0"/>
-      <geometry>
-        <mesh filename="file:///home/cameron/Project_Echo/Educational/amr_ws/src/echo_sim_v1/meshes/caster_wheel_link.STL"/>
-      </geometry>
-    </collision>
-  </link>
-  <joint name="base_link_to_caster_wheel" type="fixed">
-    <origin xyz="0.07 0.008 0" rpy="1.5708 -1.2948 3.1416"/>
-    <parent link="base_link"/>
-    <child link="caster_wheel_link"/>
-    <axis xyz="0 0 0"/>
-  </joint>
-  <!-- Lidar -->
-  <link name="lidar_link">
-    <inertial>
-      <origin xyz="-2.6195E-17 -1.1719E-17 0.0097699" rpy="0 0 0"/>
-      <mass value="0.024496"/>
-      <inertia ixx="3.1849E-06" ixy="3.1764E-22" ixz="-1.8127E-23"
-               iyy="3.1849E-06" iyz="-3.5234E-23" izz="4.7979E-06"/>
-    </inertial>
-    <visual>
-      <origin xyz="0 0 0" rpy="0 0 0"/>
-      <geometry>
-        <mesh filename="file:///home/cameron/Project_Echo/Educational/amr_ws/src/echo_sim_v1/meshes/lidar_link.STL"/>
+        <cylinder radius="0.05" length="0.04"/>
       </geometry>
       <material name="dark_grey"/>
     </visual>
     <collision>
-      <origin xyz="0 0 0" rpy="0 0 0"/>
       <geometry>
-        <mesh filename="file:///home/cameron/Project_Echo/Educational/amr_ws/src/echo_sim_v1/meshes/lidar_link.STL"/>
+        <cylinder radius="0.05" length="0.04"/>
       </geometry>
     </collision>
+    <xacro:inertial_cylinder mass="0.1" length="0.04" radius="0.05">
+      <origin xyz="0 0 0" rpy="0 0 0"/>
+    </xacro:inertial_cylinder>
   </link>
-  <joint name="base_link_to_lidar" type="fixed">
-    <origin xyz="0 -0.05 0" rpy="1.5708 0.30388 0"/>
+  <gazebo reference="left_wheel">
+    <material>Gazebo/DarkGrey</material>
+  </gazebo>
+  <!-- Right Wheel -->
+  <joint name="right_wheel_joint" type="continuous">
     <parent link="base_link"/>
-    <child link="lidar_link"/>
-    <axis xyz="0 0 0"/>
+    <child link="right_wheel"/>
+    <origin xyz="-0.07 -0.175 0" rpy="${pi/2} 0 0"/>
+    <axis xyz="0 0 1"/> <!-- made consistent -->
   </joint>
-  <!-- Camera  -->
-  <link name="camera_link">
-    <inertial>
-      <origin xyz="0.0024702 4.5609E-18 -6.9389E-18" rpy="0 0 0"/>
-      <mass value="0.00094737"/>
-      <inertia ixx="5.0737E-08" ixy="5.1013E-24" ixz="5.311E-25"
-               iyy="6.9275E-09" iyz="7.8632E-15" izz="4.7598E-08"/>
-    </inertial>
+  <link name="right_wheel">
     <visual>
-      <origin xyz="0 0 0" rpy="0 0 0"/>
       <geometry>
-        <mesh filename="file:///home/cameron/Project_Echo/Educational/amr_ws/src/echo_sim_v1/meshes/camera_link.STL"/>
+        <cylinder radius="0.05" length="0.04"/>
       </geometry>
       <material name="dark_grey"/>
     </visual>
     <collision>
-      <origin xyz="0 0 0" rpy="0 0 0"/>
       <geometry>
-        <mesh filename="file:///home/cameron/Project_Echo/Educational/amr_ws/src/echo_sim_v1/meshes/camera_link.STL"/>
+        <cylinder radius="0.05" length="0.04"/>
       </geometry>
     </collision>
+    <xacro:inertial_cylinder mass="0.1" length="0.04" radius="0.05">
+      <origin xyz="0 0 0" rpy="0 0 0"/>
+    </xacro:inertial_cylinder>
   </link>
-  <joint name="base_link_to_camera" type="fixed">
-    <origin xyz="0.1 -0.049 0" rpy="1.5708 0 0"/>
-    <parent link="base_link"/>
-    <child link="camera_link"/>
-    <axis xyz="0 0 0"/>
+  <gazebo reference="right_wheel">
+    <material>Gazebo/DarkGrey</material>
+  </gazebo>
+  <!-- Caster Wheel -->
+  <joint name="caster_wheel_joint" type="fixed">
+    <parent link="chassis"/>
+    <child link="caster_wheel"/>
+    <origin xyz="0.285 0 0"/>
   </joint>
+  <link name="caster_wheel">
+    <visual>
+      <geometry>
+        <sphere radius="0.05"/>
+      </geometry>
+      <material name="dark_grey"/>
+    </visual>
+    <collision>
+      <geometry>
+        <sphere radius="0.05"/>
+      </geometry>
+    </collision>
+    <xacro:inertial_sphere mass="0.1" radius="0.05">
+      <origin xyz="0 0 0" rpy="0 0 0"/>
+    </xacro:inertial_sphere>
+  </link>
+  <gazebo reference="caster_wheel">
+    <material>Gazebo/Grey</material>
+    <mu1 value="0.001"/>
+    <mu2 value="0.001"/>
+  </gazebo>
+<joint name="laser_joint" type="fixed">
+        <parent link="chassis"/>
+        <child link="laser_frame"/>
+        <origin xyz="0.2 0 0.15" rpy="0 0 0"/>
+    </joint>
+    <link name="laser_frame">
+        <visual>
+            <geometry>
+                <cylinder radius="0.04" length="0.05"/>
+            </geometry>
+            <material name="silver"/>
+        </visual>
+        <collision>
+            <geometry>
+                <cylinder radius="0.04" length="0.05"/>
+            </geometry>
+        </collision>
+        <xacro:inertial_cylinder mass="0.1" length="0.05" radius="0.04">
+            <origin xyz="0 0 0" rpy="0 0 0"/>
+        </xacro:inertial_cylinder>
+    </link>
+    <gazebo reference="lidar_frame">
+        <material>Gazebo/Grey</material>
+    </gazebo>
 </robot>

File: install/echo_sim_v1/share/echo_sim_v1/urdf/materials.xacro (robot description, xacro)
@@ -17,3 +17,12 @@
   <color rgba="0.2 0.2 0.2 1.0"/>
 </material>
+<material name="white">
+  <color rgba="1 1 1 1" />
+</material>
+<material name="orange">
+  <color rgba="1 0.3 0.1 1"/>
+</material>
+<material name="blue">
+  <color rgba="0.2 0.2 1 1"/>
+</material>
 </robot>

Commit message: lots of changes

File: install/echo_sim_v1/share/echo_sim_v1/urdf/echo_v1.urdf.xacro (robot description, xacro)
@@ -10,4 +10,6 @@
 <!-- Include lidar xacro -->
   <xacro:include filename="/home/cameron/Project_Echo/Educational/amr_ws/src/echo_sim_v1/urdf/lidar.xacro"/>
+<!-- Include camera xacro -->
+  <!-- <xacro:include filename="/home/cameron/Project_Echo/Educational/amr_ws/src/echo_sim_v1/urdf/camera.xacro"/> -->
   <!-- Inertia Macros -->
   <xacro:macro name="inertial_sphere" params="mass radius *origin">
@@ -149,9 +151,10 @@
     <mu2 value="0.001"/>
   </gazebo>
+<!-- Lidar -->
 <joint name="laser_joint" type="fixed">
         <parent link="chassis"/>
         <child link="laser_frame"/>
         <origin xyz="0.2 0 0.15" rpy="0 0 0"/>
-    </joint>
+</joint>
     <link name="laser_frame">
         <visual>
@@ -170,6 +173,28 @@
         </xacro:inertial_cylinder>
     </link>
-    <gazebo reference="lidar_frame">
+    <gazebo reference="laser_frame">
         <material>Gazebo/Grey</material>
     </gazebo>
+  <!-- Camera -->
+  <!-- <joint name="camera_joint" type="fixed">
+        <child link="camera_link"/>
+        <origin xyz="0.4 0 0.15" rpy="0 0 0"/>
+  </joint>
+  <link name="camera_link">
+      <visual>
+        <geometry>
+          <box size="0.015 0.03 0.03"/>
+        </geometry>
+        <material name="silver"/>
+      </visual>
+  </link>
+  <joint name="camera_optical_joint" type="fixed">
+        <parent link="camera_link"/>
+        <child link="camera_link_optical"/>
+        <origin xyz="0 0 0" rpy="${-pi/2} 0 ${-pi/2}"/>
+  </joint>
+  <link name="camera_link_optical"></link>
+  <gazebo reference="camera_link">
+    <material>Gazebo/Grey</material>
+  </gazebo> -->
 </robot>

File: install/echo_sim_v1/share/echo_sim_v1/urdf/lidar.xacro (robot description, xacro)
@@ -1,3 +1,30 @@
 <?xml version="1.0"?>
 <robot xmlns:xacro="http://ros.org/wiki/xacro">
+<gazebo reference="laser_frame">
+        <sensor name="laser" type="ray">
+            <pose> 0 0 0 0 0 0 </pose>
+            <visualize>true</visualize> <!-- Visualize in in gazebo -->
+            <update_rate>10</update_rate> <!-- sensor is updated 10x per second -->
+            <ray>
+                <scan>
+                    <horizontal>          <!-- Scans horizontally with the following parameters-->
+                        <samples>360</samples>
+                        <min_angle>-3.14</min_angle>
+                        <max_angle>3.14</max_angle>
+                    </horizontal>
+                </scan>
+                <range>
+                    <min>0.3</min>
+                    <max>12</max>
+                </range>
+            </ray>
+            <plugin name="laser_controller" filename="libgazebo_ros_ray_sensor.so">
+                <ros>
+                    <argument>~/out:=scan</argument>  <!-- Publish to the ROS topic scan -->
+                </ros>
+                <output_type>sensor_msgs/LaserScan</output_type> <!-- Publish as laser scan message -->
+                <frame_name>laser_frame</frame_name>
+            </plugin>
+        </sensor>
+    </gazebo>
 </robot>

Commit message: implemented SLAM

File: install/echo_sim_v1/share/echo_sim_v1/urdf/echo_v1.urdf.xacro (robot description, xacro)
@@ -45,4 +45,11 @@
   <!-- Base link (empty root) -->
   <link name="base_link"/>
+  <!-- Base Footprint Link -->
+  <joint name="base_footprint_joint" type="fixed">
+    <parent link="base_link"/>
+    <child link="base_footprint"/>
+    <origin xyz="0 0 0" rpy="0 0 0"/>
+  </joint>
+  <link name="base_footprint"/>
   <!-- Chassis -->
   <joint name="chassis_joint" type="fixed">
