Commit message: implemented nav2

File: src/echo_sim_v1/urdf/echo_v1.urdf.xacro (robot description, xacro)
@@ -83,9 +83,10 @@
     <parent link="base_link"/>
     <child link="left_wheel"/>
-    <origin xyz="-0.07 0.175 0" rpy="-${pi/2} 0 0"/>
-    <axis xyz="0 0 1"/>
+    <origin xyz="-0.07 0.175 0" rpy="0 0 0"/>
+    <axis xyz="0 1 0"/>
   </joint>
   <link name="left_wheel">
     <visual>
+      <origin xyz="0 0 0" rpy="${pi/2} 0 0"/>
       <geometry>
         <cylinder radius="0.05" length="0.04"/>
@@ -94,4 +95,5 @@
     </visual>
     <collision>
+      <origin xyz="0 0 0" rpy="${pi/2} 0 0"/>
       <geometry>
         <cylinder radius="0.05" length="0.04"/>
@@ -109,9 +111,10 @@
     <parent link="base_link"/>
     <child link="right_wheel"/>
-    <origin xyz="-0.07 -0.175 0" rpy="${pi/2} 0 0"/>
-    <axis xyz="0 0 1"/> <!-- made consistent -->
+    <origin xyz="-0.07 -0.175 0" rpy="0 0 0"/>
+    <axis xyz="0 1 0"/>
   </joint>
   <link name="right_wheel">
     <visual>
+      <origin xyz="0 0 0" rpy="${pi/2} 0 0"/>
       <geometry>
         <cylinder radius="0.05" length="0.04"/>
@@ -120,4 +123,5 @@
     </visual>
     <collision>
+      <origin xyz="0 0 0" rpy="${pi/2} 0 0"/>
       <geometry>
         <cylinder radius="0.05" length="0.04"/>
